Commit message: articulated

File: description/clibo_mini.xacro (robot description, xacro)
@@ -17,4 +17,7 @@
         <color rgba="1 0 0 1"/>
     </material>
+    <material name="silver">
+        <color rgba="0.7725490196078432 0.788235294117647 0.7803921568627451 1.0"/>
+    </material>
     <!-- BASE LINK -->
     <link name="base_link">
@@ -28,13 +31,13 @@
     <link name="base_footprint">
     </link>
-    <!-- CHASSIS LINK -->
-    <joint name="chassis_joint" type="fixed">
-        <parent link="base_link"/>
-        <child link="chassis"/>
+    <!-- BOTTOM BOX LINK -->
+    <joint name="bottom_box_joint" type="fixed">
+        <parent link="base_link"/>
+        <child link="bottom_box"/>
         <origin xyz="-0.15 0 0"/>
     </joint>
-    <link name="chassis">
-        <visual>
-            <origin xyz="0.15 0 0.075"/>
+    <link name="bottom_box">
+        <visual>
+            <origin xyz="0.15 0 0.0375"/>
             <geometry>
                 <box size="0.3 0.3 0.15"/>
@@ -43,5 +46,5 @@
         </visual>
         <collision>
-            <origin xyz="0.15 0 0.075"/>
+            <origin xyz="0.15 0 0.0375"/>
             <geometry>
                 <box size="0.3 0.3 0.15"/>
@@ -49,12 +52,66 @@
         </collision>
         <xacro:inertial_box mass="0.5" x="0.3" y="0.3" z="0.15">
-            <origin xyz="0.15 0 0.075" rpy="0 0 0"/>
+            <origin xyz="0.15 0 0.0375" rpy="0 0 0"/>
         </xacro:inertial_box>
     </link>
-    <gazebo reference="chassis">
+    <gazebo reference="bottom_box">
+        <material>Gazebo/White</material>
+    </gazebo>
+    <!-- MIDDLE BOX LINK -->
+    <joint name="middle_box_joint" type="fixed">
+        <parent link="base_link"/>
+        <child link="middle_box"/>
+        <origin xyz="0 0 0.15"/>
+    </joint>
+    <link name="middle_box">
+        <visual>
+            <origin xyz="0 0 0.15"/>
+            <geometry>
+                <box size="0.15 0.15 0.0375"/>
+            </geometry>
+            <material name ="white"/>
+        </visual>
+        <collision>
+            <origin xyz="0 0 0.15"/>
+            <geometry>
+                <box size="0.15 0.15 0.0375"/>
+            </geometry>
+        </collision>
+        <xacro:inertial_box mass="0.5" x="0.15" y="0.15" z="0.0375">
+            <origin xyz="0 0 0.15" rpy="0 0 0"/>
+        </xacro:inertial_box>
+    </link>
+    <gazebo reference="middle_box">
+        <material>Gazebo/White</material>
+    </gazebo>
+    <!-- UPPER BOX LINK -->
+    <joint name="upper_box_joint" type="fixed">
+        <parent link="base_link"/>
+        <child link="upper"/>
+        <origin xyz="-0.15 0 0"/>
+    </joint>
+    <link name="upper_box">
+        <visual>
+            <origin xyz="0 0 0.1875"/>
+            <geometry>
+                <box size="0.3 0.3 0.3"/>
+            </geometry>
+            <material name ="white"/>
+        </visual>
+        <collision>
+            <origin xyz="0.15 0 0.1875"/>
+            <geometry>
+                <box size="0.3 0.3 0.3"/>
+            </geometry>
+        </collision>
+        <xacro:inertial_box mass="0.5" x="0.3" y="0.3" z="0.3">
+            <origin xyz="0 0 0.1875" rpy="0 0 0"/>
+        </xacro:inertial_box>
+    </link>
+    <gazebo reference="upper_box">
         <material>Gazebo/White</material>
     </gazebo>
     <!-- OUTER CASE LINK-->
-    <joint name="outer_case_joint" type="fixed">
+  <!--  <joint name="outer_case_joint" type="fixed">
         <parent link="base_link"/>
         <child link="outer_case"/>
@@ -101,5 +158,5 @@
         <collision>
             <geometry>
-                <sphere radius="0.05"/>
+                <cylinder radius="0.05" length="0.04"/>
             </geometry>
         </collision>
@@ -127,9 +184,9 @@
         <collision>
             <geometry>
-                <sphere radius="0.05"/>
-            </geometry>
+                <cylinder radius="0.05" length="0.04"/>
+            </geometry>robot urdf stl files
         </collision>
         <xacro:inertial_cylinder mass="0.1" length="0.04" radius="0.05">
-            <origin xyz="0 0 0 " rpy="0 0 0"/>
+            <origin xyz="0 0 0 " rpy="0 0 0"/>robot urdf stl files
         </xacro:inertial_cylinder>
     </link>
@@ -246,3 +303,3 @@
         <mu2 value="0.001"/>
     </gazebo>
-</robot>
+</robot>-->

File: description/gazebo_control.xacro (robot description, xacro)
@@ -2,5 +2,5 @@
 <robot xmlns:xacro="http://www.ros.org/wiki/xacro">
     <gazebo>
-        <plugin name="diff_drive" filename="libgazebo_ros_diffdrive.so">
+        <plugin name="diff_drive" filename="libgazebo_ros_diff_drive.so">
             <!-- Wheel Information -->
             <left_joint>left_wheel_joint</left_joint>

File: description/inertial_macros.xacro (robot description, xacro)
@@ -30,3 +30,12 @@
         </inertial>
     </xacro:macro>
+    <xacro:macro name="inertial_doughnut" params="mass x y z *origin">
+        <inertial>
+            <xacro:insert_block name="origin"/>
+            <mass value="${mass}" />
+            <inertia ixx="${(1/12) * mass * (y*y + z*z)}" ixy="0.0" ixz="0.0"
+                    iyy="${(1/12) * mass * (x*x + z*z)}" iyz="0.0"
+                    izz="${(1/12) * mass * (x*x + y*y)}" />
+        </inertial>
+    </xacro:macro>
 </robot>

File: description/robot.urdf.xacro (robot description, xacro)
@@ -1,5 +1,14 @@
 <?xml version="1.0"?>
-<robot xmlns:xacro="http://www.ros.org/wiki/xacro"  name="robot">
-    <xacro:include filename="robot_core.xacro"/>
-    <xacro:include filename="gazebo_control.xacro"/>
+<robot xmlns:xacro="http://www.ros.org/wiki/xacro"  name="clibo">
+    <xacro:arg name="use_ros2_control" default="true" />
+    <xacro:arg name="sim_mode" default="false" />
+    <xacro:include filename="robot_core.xacro" />
+    <xacro:if value="$(arg use_ros2_control)">
+        <xacro:include filename="ros2_control.xacro" />
+    </xacro:if>
+    <xacro:unless value="$(arg use_ros2_control)">
+        <xacro:include filename="gazebo_control.xacro" />
+    </xacro:unless>
+    <xacro:include filename="lidar.xacro" />
+    <xacro:include filename="face.xacro" />
 </robot>
